File: TuksBaja Electrical System.kicad_sch (KiCad schematic)
At the start: 7 parts, among them U1 LM2596S-ADJ

Commit message: removed dubious power flags
Changed lines of the file:
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@@
-	)
-	(junction
-		(at 134.62 60.96)
-		(diameter 0)
-		(color 0 0 0 0)
-	)
-	(junction
-		(at 119.38 50.8)
-		(diameter 0)
-		(color 0 0 0 0)
 	)
 	(junction
@@
 	(wire
 		(pts
-			(xy 116.84 50.8) (xy 119.38 50.8)
+			(xy 116.84 50.8) (xy 134.62 50.8)
 		)
 		(stroke
@@
 	(wire
 		(pts
-			(xy 119.38 50.8) (xy 134.62 50.8)
-		)
-		(stroke
-			(width 0)
-			(type default)
-		)
-	)
-	(wire
-		(pts
 			(xy 69.85 60.96) (xy 59.69 60.96)
 		)
@@
 			(width 0)
 			(type default)
-		)
-	)
-	(symbol
-		(lib_id "power:PWR_FLAG")
-		(at 119.38 50.8 0)
-		(unit 1)
-		(exclude_from_sim no)
-		(in_bom yes)
-		(on_board yes)
-		(dnp no)
-		(fields_autoplaced yes)
-		(property "Reference" "#FLG01"
-			(at 119.38 48.895 0)
-			(effects
-				(font
-					(size 1.27 1.27)
-				)
-				(hide yes)
-			)
-		)
-		(property "Value" "PWR_FLAG"
-			(at 119.38 45.72 0)
-			(effects
-				(font
-					(size 1.27 1.27)
-				)
-			)
-		)
-		(property "Footprint" ""
-			(at 119.38 50.8 0)
-			(effects
-				(font
-					(size 1.27 1.27)
-				)
-				(hide yes)
-			)
-		)
-		(property "Datasheet" "~"
-			(at 119.38 50.8 0)
-			(effects
-				(font
-					(size 1.27 1.27)
-				)
-				(hide yes)
-			)
-		)
-		(property "Description" "Special symbol for telling ERC where power comes from"
-			(at 119.38 50.8 0)
-			(effects
-				(font
-					(size 1.27 1.27)
-				)
-				(hide yes)
-			)
-		)
-		(pin "1"
-		)
-		(instances
-			(project ""
-				(path "/32101482-20ad-4a29-9fb3-a9077501af62"
-					(reference "#FLG01")
-					(unit 1)
-				)
-			)
 		)
 	)
@@
 					(unit 1)
 				)
-			)
-		)
-	)
-	(symbol
-		(lib_id "power:PWR_FLAG")
-		(at 134.62 60.96 0)
-		(unit 1)
-		(exclude_from_sim no)
-		(in_bom yes)
-		(on_board yes)
-		(dnp no)
-		(fields_autoplaced yes)
-		(property "Reference" "#FLG03"
-			(at 134.62 59.055 0)
-			(effects
-				(font
-					(size 1.27 1.27)
-				)
-				(hide yes)
-			)
-		)
-		(property "Value" "PWR_FLAG"
-			(at 134.62 55.88 0)
-			(effects
-				(font
-					(size 1.27 1.27)
-				)
-			)
-		)
-		(property "Footprint" ""
-			(at 134.62 60.96 0)
-			(effects
-				(font
-					(size 1.27 1.27)
-				)
-				(hide yes)
-			)
-		)
-		(property "Datasheet" "~"
-			(at 134.62 60.96 0)
-			(effects
-				(font
-					(size 1.27 1.27)
-				)
-				(hide yes)
-			)
-		)
-		(property "Description" "Special symbol for telling ERC where power comes from"
-			(at 134.62 60.96 0)
-			(effects
-				(font
-					(size 1.27 1.27)
-				)
-				(hide yes)
-			)
-		)
-		(pin "1"
-		)
-		(instances
-			(project ""
-				(path "/32101482-20ad-4a29-9fb3-a9077501af62"
-					(reference "#FLG03")
-					(unit 1)
-				)

Commit message: added hall effect sensor
Parts:
- added A1: Arduino_UNO_R3, Module:Arduino_UNO_R3, symbol MCU_Module:Arduino_UNO_R3
- added Battery: 12V, symbol Device:Battery
- added HallEffect: A1104xLH, Package_TO_SOT_SMD:SOT-23W, symbol Sensor_Magnetic:A1104xLH
- R2: value 3k -> ?
- renumbered U1 to BuckConverter
Connections:
- net +12V: now also Battery.1 (+)
- net GND: now also A1.29 (GND), A1.6 (GND), A1.7 (GND), HallEffect.3 (GND)
- net +5V renamed +7.5V
- net +7.5V: now also A1.8 (VIN)
- new net: A1.5 (+5V), HallEffect.1 (V_{CC})
- new net: A1.9 (A0), HallEffect.2 (V_{OUT})
- new net GNDPWR: Battery.2 (-)
Other:
- note added: "Main Bus"
- note added: "Signal and Control"
- note added: "Signal and Control Power Rail"
- note removed: "Power Supply"
- moved on the sheet: BuckConverter, C_IN1, C_OUT1, D1, L1, R1, R2

Commit message: added sensor filtering and amplification
Parts:
- removed A1: Arduino_UNO_R3, Module:Arduino_UNO_R3, symbol MCU_Module:Arduino_UNO_R3
- removed HallEffect: A1104xLH, Package_TO_SOT_SMD:SOT-23W, symbol Sensor_Magnetic:A1104xLH
- added C1: C, symbol Device:C
- added OP_AMP, U1: TL064, symbol Amplifier_Operational:TL064
- added R3, R4, R5: R_US, symbol Device:R_US
- added U2: A1104xLH, Package_TO_SOT_SMD:SOT-23W, symbol Sensor_Magnetic:A1104xLH
Connections:
- net GND: now also C1.2, U1.11 (V-), U2.3 (GND)
- new net: OP_AMP.3 (+), R5.1
- new net: OP_AMP.1, R5.2
- new net: C1.1, R3.2, R4.2
- new net: OP_AMP.2 (-), R3.1
- new net: R4.1, U2.2 (V_{OUT})
- new net +5V: U1.4 (V+), U2.1 (V_{CC})
Other:
- note added: "Low Voltage Power Rail"
- note removed: "Signal and Control"
- note removed: "Signal and Control Power Rail"

Commit message: critical modifications
Parts:
- removed Battery: 12V, symbol Device:Battery
- removed OP_AMP, U1: TL064, symbol Amplifier_Operational:TL064
- removed R3, R4, R5: R_US, symbol Device:R_US
- added C2: 0.1u, symbol Device:C
- added R3, R4: 100k, symbol Device:R
- added U1, U5: LM358, symbol Amplifier_Operational:LM358
- added U3: ESP32-S3-WROOM-1, RF_Module:ESP32-S3-WROOM-1, symbol RF_Module:ESP32-S3-WROOM-1
- added U4: A1104xLH, Package_TO_SOT_SMD:SOT-23W, symbol Sensor_Magnetic:A1104xLH
- C1: value C -> 0.1u
Connections:
- net +5V: now also C1.1, C2.1, U4.1 (V_{CC})
- net GND: now also C2.2, R3.1, R4.1, U1.3 (+), U1.4 (V-), U4.3 (GND), U5.3 (+), U5.4 (V-)
- net at U2.2 (V_{OUT}): now also U1.2 (-)
- net +7.5V renamed +3.3V
- new net: U3.1 (GND), U3.40 (GND), U3.41 (GND)
- new net: U4.2 (V_{OUT}), U5.2 (-)
- new net RL_WS: R3.2, U1.1
- new net RR_WS: R4.2, U5.1
Other:
- note added: "0.1 uF capacitor for decoupling"
- note added: "Rear Left Wheel Speed"
- note added: "Rear Right Wheel Speed"
- note added: "Step Down Converter"
- note removed: "Low Voltage Power Rail"
- note removed: "Main Bus"
- moved on the sheet: BuckConverter, C_IN1, C_OUT1, D1, L1, R1, R2, U2
